Commit message: added MoveIt Config

File: armbot_description/onshape_to_robot/armbot/robot.urdf (robot description, URDF)
Before this commit: robot armbot, 18 links, 17 joints
Joints:
- joint 2020_To_HebiRotor2020: limit effort=1 velocity=20 -> effort=1 velocity=20.0
- joint 2040_To_HebiStatorNormal: limit effort=1 velocity=20 -> effort=1 velocity=20.0
- joint Base2040_To_Base_HebiRotor2020: limit effort=1 velocity=20 -> effort=1 velocity=20.0
- joint Base_HebiRotor2020_Base2020: limit effort=1 velocity=20 -> effort=1 velocity=20.0
- joint Base_HebiRotor2020_Base2020_2: limit effort=1 velocity=20 -> effort=1 velocity=20.0
- joint Base_HebiRotor2020_Base2040_2: limit effort=1 velocity=20 -> effort=1 velocity=20.0
- joint DynaMount_To_2020: limit effort=1 velocity=20 -> effort=1 velocity=20.0
- joint DynaRotor_To_Dynamixel_J2: limit lower=-3.141592653589793116 upper=1.570796326794896558 effort=1 velocity=20 -> lower=-3.141592653589793116 upper=1.570796326794896558 effort=1 velocity=20.0
- joint DynaRotor_To_Dynamixel_J3: limit lower=-50.265482457436689856 upper=50.265482457436689856 effort=1 velocity=20 -> lower=-50.265482457436689856 upper=50.265482457436689856 effort=1 velocity=20.0
- joint DynaRotor_to_DynaMount: limit effort=1 velocity=20 -> effort=1 velocity=20.0
- joint HebiRotor2020_To_HebiBase: limit effort=1 velocity=20 -> effort=1 velocity=20.0
- joint HebiRotor2020_to_J1_Hebi: limit effort=1 velocity=20 -> effort=1 velocity=20.0
- joint HebiStatorRightAngle_To_2040: limit effort=1 velocity=20 -> effort=1 velocity=20.0
- joint Hebi_Base_Stator_To_HebiStatorNormal: limit effort=1 velocity=20 -> effort=1 velocity=20.0
- joint Hebi_J1_Stator_To_HebiStatorRightAngle: limit effort=1 velocity=20 -> effort=1 velocity=20.0
- joint Hebi_Rotor_Base: limit lower=-6.283185307179586232 upper=6.283185307179586232 effort=1 velocity=20 -> lower=-6.283185307179586232 upper=6.283185307179586232 effort=1 velocity=20.0
- joint Hebi_Rotor_J1: limit lower=-2.356194490192344837 upper=2.356194490192344837 effort=1 velocity=20 -> lower=-2.356194490192344837 upper=2.356194490192344837 effort=1 velocity=20.0

Commit message: dynamixel mostly working

File: armbot_description/onshape_to_robot/armbot/robot.urdf (robot description, URDF)
Before this commit: robot armbot, 18 links, 17 joints
Links:
- link hebi_stator_: mass 0.29483503919999992648 -> 0.29483503920000003751
- link hebi_stator__2: mass 0.29483503919999992648 -> 0.29483503920000003751
Joints:
- joint 2020_To_HebiRotor2020: limit effort=1 velocity=20.0 -> effort=1 velocity=20
- joint 2040_To_HebiStatorNormal: limit effort=1 velocity=20.0 -> effort=1 velocity=20
- joint Base2040_To_Base_HebiRotor2020: limit effort=1 velocity=20.0 -> effort=1 velocity=20
- joint Base_HebiRotor2020_Base2020: limit effort=1 velocity=20.0 -> effort=1 velocity=20
- joint Base_HebiRotor2020_Base2020_2: limit effort=1 velocity=20.0 -> effort=1 velocity=20
- joint Base_HebiRotor2020_Base2040_2: limit effort=1 velocity=20.0 -> effort=1 velocity=20
- joint DynaMount_To_2020: limit effort=1 velocity=20.0 -> effort=1 velocity=20
- joint DynaRotor_To_Dynamixel_J2: limit lower=-3.141592653589793116 upper=1.570796326794896558 effort=1 velocity=20.0 -> lower=0 upper=4.712388980384689674 effort=1 velocity=20; origin xyz=0.0080000000000000001665 5.5511151231257827021e-17 0.00025000002471399496162 rpy=3.5599014307809674267e-15 -8.813389537416573132e-15 1.5707963267948992225 -> xyz=0.0080000000000000088402 5.5511151231257827021e-17 0.00025000002471403659499 rpy=1.4592157403991824048e-15 -2.0114719705239952011e-16 -2.1693674893577824649e-30
- joint DynaRotor_To_Dynamixel_J3: limit lower=-50.265482457436689856 upper=50.265482457436689856 effort=1 velocity=20.0 -> lower=-50.265482457436689856 upper=50.265482457436689856 effort=1 velocity=20; origin xyz=0.019000000000000016875 -0.023999999999999990091 -0.019000000000000030753 rpy=1.5707963267981290834 -1.5707105036825337319 1.5707963268983915484 -> xyz=0.019000000000000058509 -0.024000000000000021316 -0.019000000000000030753 rpy=1.5707963267999121015 -1.5707513548487626043 1.570796326804927201
- joint DynaRotor_to_DynaMount: limit effort=1 velocity=20.0 -> effort=1 velocity=20; origin xyz=0.023843291201925909117 0.0079829788319448410916 -0.008999999999999980238 rpy=3.551440358039829389e-17 8.3266726846887307526e-17 -1.570796326794896558 -> xyz=0.023843291201925853606 0.0079829788319448358874 -0.0089999999999999524825 rpy=3.5514403580398096675e-17 8.326672684688884827e-17 -1.570796326794896558
- joint HebiRotor2020_To_HebiBase: limit effort=1 velocity=20.0 -> effort=1 velocity=20
- joint HebiRotor2020_to_J1_Hebi: limit effort=1 velocity=20.0 -> effort=1 velocity=20
- joint HebiStatorRightAngle_To_2040: limit effort=1 velocity=20.0 -> effort=1 velocity=20
- joint Hebi_Base_Stator_To_HebiStatorNormal: limit effort=1 velocity=20.0 -> effort=1 velocity=20
- joint Hebi_J1_Stator_To_HebiStatorRightAngle: limit effort=1 velocity=20.0 -> effort=1 velocity=20
- joint Hebi_Rotor_Base: limit lower=-6.283185307179586232 upper=6.283185307179586232 effort=1 velocity=20.0 -> lower=-6.283185307179586232 upper=6.283185307179586232 effort=1 velocity=20
- joint Hebi_Rotor_J1: limit lower=-2.356194490192344837 upper=2.356194490192344837 effort=1 velocity=20.0 -> lower=-2.356194490192344837 upper=2.356194490192344837 effort=1 velocity=20

Commit message: mostly there for showcase

File: armbot_description/onshape_to_robot/armbot/robot.urdf (robot description, URDF)
Before this commit: robot armbot, 18 links, 17 joints
Joints:
- joint DynaRotor_To_Dynamixel_J2: limit lower=0 upper=4.712388980384689674 effort=1 velocity=20 -> lower=0 upper=4.712388980384689674 effort=1 velocity=4
- joint DynaRotor_To_Dynamixel_J3: limit lower=-50.265482457436689856 upper=50.265482457436689856 effort=1 velocity=20 -> lower=-10 upper=10 effort=1 velocity=4
- joint Hebi_Rotor_Base: limit lower=-6.283185307179586232 upper=6.283185307179586232 effort=1 velocity=20 -> lower=-6.283185307179586232 upper=6.283185307179586232 effort=1 velocity=3
- joint Hebi_Rotor_J1: limit lower=-2.356194490192344837 upper=2.356194490192344837 effort=1 velocity=20 -> lower=-2.356194490192344837 upper=2.356194490192344837 effort=1 velocity=0.5
